Commit message: Made some changes to the turbid water world some more, and attempted some modification to the FLSonar plugin. Still unsuccesful rendering and requiring more debugging.

File: uuv_descriptions/robots/rexrov_flsonar.xacro (robot description, xacro)
@@ -39,4 +39,7 @@
     <origin xyz="1.4 0 0.65" rpy="0 0 0"/>
   </xacro:forward_multibeam_sonar_m450_130>
+  <!--<xacro:fl_multibeam_generic namespace="$(arg namespace)" parent_link="$(arg namespace)/base_link">
+    <origin xyz="1.4 0 0.65" rpy="0 0 0"/>
+  </xacro:fl_multibeam_generic>-->
   <!-- Joint state publisher plugin -->
   <xacro:default_joint_state_publisher namespace="$(arg namespace)" update_rate="50"/>

File: uuv_sensor_plugins/uuv_sensor_ros_plugins/urdf/sonar_snippets.xacro (robot description, xacro)
@@ -142,5 +142,6 @@
     <sensor type="gpu_ray" name="sonar${suffix}">
       <pose>0 0 0 0 0 0</pose>
-      <visualize>false</visualize>
+      <!--Change value here to make sonar beams visible or not-->
+      <visualize>true</visualize>
       <update_rate>${update_rate}</update_rate>
       <ray>
@@ -201,5 +202,5 @@
       <sensor name='FLSonar' type='camera'>
         <plugin name="SonarVisual" filename="libuuv_gazebo_ros_flsonar_plugin.so" >
-            <topic>${topic}</topic>
+            <topic>rexrov/FLSonar</topic>
             <debug>1</debug>
             <link_reference>${namespace}/sonar${suffix}_link</link_reference>
