Commit message: Changed environment to use exponential fog which better mimics turbid water. Also added Kinect Depth camera to customized rexrov, simulating acoustic camera.

File: uuv_descriptions/robots/rexrov_test.xacro (robot description, xacro)
@@ -22,4 +22,7 @@
     <origin xyz="7.5 0 15" rpy="0 1.52 0"/>
   </xacro:default_camera>
+  <xacro:uw_depth_camera namespace="${namespace}" parent_link="${namespace}/base_link" suffix="depth">
+    <origin xyz="1.15 0.5 0.4" rpy="0 0.1 0"/>
+  </xacro:uw_depth_camera>
   <!-- Create the RexROV vehicle -->
   <xacro:rexrov_base

Commit message: Added fls implementation by Niels Bohr as explained in the following issue thread: https://github.com/uuvsimulator/uuv_simulator/issues/48, with the main code of the fls contained here: https://github.com/smarc-project/smarc_simulations/blob/master/smarc_gazebo_plugins/smarc_gazebo_ros_plugins/src/gazebo_ros_image_sonar.cpp. \n\n TODO: Modify FLS to be better representation (current FLS still abuses Depth cam), and integrate FLS into our project environment/requirement better

File: uuv_descriptions/robots/rexrov_test.xacro (robot description, xacro)
@@ -22,7 +22,29 @@
     <origin xyz="7.5 0 15" rpy="0 1.52 0"/>
   </xacro:default_camera>
-  <xacro:uw_depth_camera namespace="${namespace}" parent_link="${namespace}/base_link" suffix="depth">
+  <!--<xacro:uw_depth_camera namespace="${namespace}" parent_link="${namespace}/base_link" suffix="depth">
     <origin xyz="1.15 0.5 0.4" rpy="0 0.1 0"/>
-  </xacro:uw_depth_camera>
+  </xacro:uw_depth_camera>-->
+  <!--
+  <xacro:fls_camera namespace="${namespace}" parent_link="${namespace}/base_link" suffix="fls">
+    <origin xyz="1.15 0.5 0.4" rpy="0 0.3 0"/>
+  </xacro:fls_camera>
+  -->
+  <xacro:forward_looking_sonar
+      namespace="${namespace}"
+      suffix="down"
+      parent_link="${namespace}/base_link"
+      topic="forward_sonar"
+      mass="0.015"
+      update_rate="10"
+      samples="100"
+        fov="1.54719755"
+        width="260"
+        height="120">
+      <inertia ixx="0.00001" ixy="0.0" ixz="0.0" iyy="0.00001" iyz="0.0" izz="0.00001" />
+      <origin xyz="0.83 0 -0.22" rpy="0 ${0.2*pi} 0" />
+      <!--<origin xyz="1.15 0 0.4" rpy="0 0.6 0"/>-->
+      <visual>
+      </visual>
+    </xacro:forward_looking_sonar>
   <!-- Create the RexROV vehicle -->
   <xacro:rexrov_base

File: uuv_sensor_plugins/uuv_sensor_ros_plugins/urdf/sonar_snippets.xacro (robot description, xacro)
@@ -227,3 +227,60 @@
     </gazebo>
   </xacro:macro>
+  <xacro:macro name="forward_looking_sonar"
+    params="namespace suffix parent_link topic mass update_rate
+      samples fov width height *inertia *origin *visual">
+    <!-- Sensor link -->
+    <link name="${namespace}/forward_sonar${suffix}_link">
+      <inertial>
+        <xacro:insert_block name="inertia" />
+        <mass value="${mass}" />
+        <origin xyz="0 0 0" rpy="0 0 0" />
+      </inertial>
+      <visual>
+        <geometry>
+          <mesh filename="file://$(find uuv_sensor_ros_plugins)/meshes/oe14-372.dae" scale="1 1 1"/>
+        </geometry>
+      </visual>
+      <!-- <xacro:insert_block name="visual" /> -->
+      <xacro:no_collision/>
+    </link>
+    <joint name="${namespace}_forward_sonar${suffix}_joint" type="revolute">
+      <xacro:insert_block name="origin" />
+      <parent link="${parent_link}" />
+      <child link="${namespace}/forward_sonar${suffix}_link" />
+      <limit upper="0" lower="0" effort="0" velocity="0" />
+      <axis xyz="1 0 0"/>
+    </joint>
+    <gazebo reference="${namespace}/forward_sonar${suffix}_link">
+      <sensor name="${namespace}/image_sonar" type="depth">
+        <camera>
+		  <horizontal_fov>${fov}</horizontal_fov>
+          <image>
+		    <width>${width}</width>
+		    <height>${height}</height>
+            <format>R8G8B8</format>
+          </image>
+          <clip>
+            <near>0.1</near>
+            <far>17</far>
+          </clip>
+          <save enabled="true">
+            <path>/tmp/camera</path>
+          </save>
+        </camera>
+	    <plugin filename="libimage_sonar_ros_plugin.so" name="forward_sonar${suffix}_controller">
+		  <topicName>${topic}</topicName>
+          <frameName>forward_sonar${suffix}_optical_frame</frameName>
+        </plugin>
+        <always_on>true</always_on>
+	    <update_rate>${update_rate}</update_rate>
+      </sensor>
+    </gazebo>
+	<joint name="${namespace}/forward_sonar${suffix}_joint" type="fixed">
+      <origin xyz="0 0 0" rpy="${-pi/2} 0 ${-pi/2}"/>
+      <parent link="${namespace}/forward_sonar${suffix}_link"/>
+      <child link="${namespace}/forward_sonar${suffix}_optical_frame"/>
+    </joint>
+	<link name="${namespace}/forward_sonar${suffix}_optical_frame"/>
+  </xacro:macro>
 </robot>

Commit message: Disabled saving of image sonar capture to avoid storage overload. Also some recent modifications to rviz for project use.

File: uuv_descriptions/robots/rexrov_test.xacro (robot description, xacro)
@@ -42,6 +42,6 @@
         height="492">
       <inertia ixx="0.00001" ixy="0.0" ixz="0.0" iyy="0.00001" iyz="0.0" izz="0.00001" />
-      <origin xyz="0.83 0 -0.22" rpy="0 ${0.2*pi} 0" />
-      <!--<origin xyz="1.15 0 0.4" rpy="0 0.6 0"/>-->
+      <!--origin xyz="0.83 0 -0.22" rpy="0 ${0.2*pi} 0" /-->
+      <origin xyz="1.15 0 0.4" rpy="0 0.3 0"/>
       <visual>
       </visual>

File: uuv_sensor_plugins/uuv_sensor_ros_plugins/urdf/sonar_snippets.xacro (robot description, xacro)
@@ -265,5 +265,5 @@
             <far>17</far>
           </clip>
-          <save enabled="true">
+          <save enabled="false"> <!--Keeping save disabled to avoid filesystem overload -->
             <path>/tmp/camera</path>
           </save>

Commit message: Matching current changes to the ones ma de at realistic-sonar branch that uses Nils Bore's WIP FLS

File: uuv_descriptions/robots/rexrov_test.xacro (robot description, xacro)
@@ -19,10 +19,32 @@
   <xacro:include filename="$(find uuv_descriptions)/urdf/rexrov_base.xacro"/>
   <xacro:include filename="$(find uuv_descriptions)/urdf/rexrov.gazebo.xacro"/>
-  <xacro:default_camera namespace="${namespace}" parent_link="${namespace}/base_link" suffix="top">
+  <!--xacro:default_camera namespace="${namespace}" parent_link="${namespace}/base_link" suffix="top">
     <origin xyz="7.5 0 15" rpy="0 1.52 0"/>
-  </xacro:default_camera>
-  <xacro:uw_depth_camera namespace="${namespace}" parent_link="${namespace}/base_link" suffix="depth">
+  </xacro:default_camera-->
+  <!--<xacro:uw_depth_camera namespace="${namespace}" parent_link="${namespace}/base_link" suffix="depth">
     <origin xyz="1.15 0.5 0.4" rpy="0 0.1 0"/>
-  </xacro:uw_depth_camera>
+  </xacro:uw_depth_camera>-->
+  <!--
+  <xacro:fls_camera namespace="${namespace}" parent_link="${namespace}/base_link" suffix="fls">
+    <origin xyz="1.15 0.5 0.4" rpy="0 0.3 0"/>
+  </xacro:fls_camera>
+  -->
+  <xacro:forward_looking_sonar
+      namespace="${namespace}"
+      suffix="down"
+      parent_link="${namespace}/base_link"
+      topic="forward_sonar"
+      mass="0.015"
+      update_rate="40"
+      samples="100"
+        fov="1.54719755"
+        width="768"
+        height="492">
+      <inertia ixx="0.00001" ixy="0.0" ixz="0.0" iyy="0.00001" iyz="0.0" izz="0.00001" />
+      <!--origin xyz="0.83 0 -0.22" rpy="0 ${0.2*pi} 0" /-->
+      <origin xyz="1.15 0 0.4" rpy="0 0.3 0"/>
+      <visual>
+      </visual>
+    </xacro:forward_looking_sonar>
   <!-- Create the RexROV vehicle -->
   <xacro:rexrov_base
@@ -41,7 +63,7 @@
     </gazebo>
   </xacro:rexrov_base>
-  <xacro:forward_multibeam_p900 namespace="$(arg namespace)" parent_link="$(arg namespace)/base_link">
+  <!--xacro:forward_multibeam_p900 namespace="$(arg namespace)" parent_link="$(arg namespace)/base_link">
     <origin xyz="1.4 0 0.65" rpy="0 0 0"/>
-  </xacro:forward_multibeam_p900>
+  </xacro:forward_multibeam_p900-->
   <!--<xacro:fl_multibeam_generic namespace="$(arg namespace)" parent_link="$(arg namespace)/base_link">
     <origin xyz="1.4 0 0.65" rpy="0 0 0"/>

File: uuv_sensor_plugins/uuv_sensor_ros_plugins/urdf/camera_snippets.xacro (robot description, xacro)
@@ -29,5 +29,5 @@
       topic="camera"
       mass="0.1"
-      update_rate="30"
+      update_rate="60"
       hfov="1.5125"
       width="768"
@@ -57,5 +57,5 @@
   </xacro:macro>
   <xacro:macro name="uw_depth_camera" params="namespace parent_link suffix *origin">
-    <xacro:uw_camera_plugin_macro
+    <xacro:uw_depthcam_plugin_macro
       namespace="${namespace}"
       suffix="${suffix}"
@@ -71,7 +71,7 @@
       <inertia ixx="0.00001" ixy="0.0" ixz="0.0" iyy="0.00001" iyz="0.0" izz="0.00001" />
       <xacro:insert_block name="origin" />
-    </xacro:uw_camera_plugin_macro>
-  </xacro:macro>
-  <xacro:macro name="uw_camera_plugin_macro"
+    </xacro:uw_depthcam_plugin_macro>
+  </xacro:macro>
+  <xacro:macro name="uw_depthcam_plugin_macro"
     params="namespace suffix parent_link topic mass update_rate
       hfov width height stddev scale

File: uuv_sensor_plugins/uuv_sensor_ros_plugins/urdf/sonar_snippets.xacro (robot description, xacro)
@@ -227,3 +227,60 @@
     </gazebo>
   </xacro:macro>
+  <xacro:macro name="forward_looking_sonar"
+    params="namespace suffix parent_link topic mass update_rate
+      samples fov width height *inertia *origin *visual">
+    <!-- Sensor link -->
+    <link name="${namespace}/forward_sonar${suffix}_link">
+      <inertial>
+        <xacro:insert_block name="inertia" />
+        <mass value="${mass}" />
+        <origin xyz="0 0 0" rpy="0 0 0" />
+      </inertial>
+      <visual>
+        <geometry>
+          <mesh filename="file://$(find uuv_sensor_ros_plugins)/meshes/oe14-372.dae" scale="1 1 1"/>
+        </geometry>
+      </visual>
+      <!-- <xacro:insert_block name="visual" /> -->
+      <xacro:no_collision/>
+    </link>
+    <joint name="${namespace}_forward_sonar${suffix}_joint" type="revolute">
+      <xacro:insert_block name="origin" />
+      <parent link="${parent_link}" />
+      <child link="${namespace}/forward_sonar${suffix}_link" />
+      <limit upper="0" lower="0" effort="0" velocity="0" />
+      <axis xyz="1 0 0"/>
+    </joint>
+    <gazebo reference="${namespace}/forward_sonar${suffix}_link">
+      <sensor name="${namespace}/image_sonar" type="depth">
+        <camera>
+          <horizontal_fov>${fov}</horizontal_fov>
+          <image>
+            <width>${width}</width>
+            <height>${height}</height>
+            <format>R8G8B8</format>
+          </image>
+          <clip>
+            <near>0.1</near>
+            <far>17</far>
+          </clip>
+          <save enabled="false"> <!--Keeping save disabled to avoid filesystem overload -->
+            <path>/tmp/camera</path>
+          </save>
+        </camera>
+	      <plugin filename="libimage_sonar_ros_plugin.so" name="forward_sonar${suffix}_controller">
+		      <topicName>${topic}</topicName>
+          <frameName>forward_sonar${suffix}_optical_frame</frameName>
+        </plugin>
+        <always_on>true</always_on>
+	      <update_rate>${update_rate}</update_rate>
+      </sensor>
+    </gazebo>
+	<joint name="${namespace}/forward_sonar${suffix}_joint" type="fixed">
+      <origin xyz="0 0 0" rpy="${-pi/2} 0 ${-pi/2}"/>
+      <parent link="${namespace}/forward_sonar${suffix}_link"/>
+      <child link="${namespace}/forward_sonar${suffix}_optical_frame"/>
+    </joint>
+	<link name="${namespace}/forward_sonar${suffix}_optical_frame"/>
+  </xacro:macro>
 </robot>

Commit message: Deleted extra xacro-s that might get unnecessarily referenced by catkin when building. Current branch works fine but might sometimes have Gazebo GUI or RViz 'process died' error which requires a re-launch. Fix to this stability is required as part of TODO list

File: uuv_descriptions/robots/rexrov_test.xacro (robot description, xacro)
@@ -19,15 +19,4 @@
   <xacro:include filename="$(find uuv_descriptions)/urdf/rexrov_base.xacro"/>
   <xacro:include filename="$(find uuv_descriptions)/urdf/rexrov.gazebo.xacro"/>
-  <!--xacro:default_camera namespace="${namespace}" parent_link="${namespace}/base_link" suffix="top">
-    <origin xyz="7.5 0 15" rpy="0 1.52 0"/>
-  </xacro:default_camera-->
-  <!--<xacro:uw_depth_camera namespace="${namespace}" parent_link="${namespace}/base_link" suffix="depth">
-    <origin xyz="1.15 0.5 0.4" rpy="0 0.1 0"/>
-  </xacro:uw_depth_camera>-->
-  <!--
-  <xacro:fls_camera namespace="${namespace}" parent_link="${namespace}/base_link" suffix="fls">
-    <origin xyz="1.15 0.5 0.4" rpy="0 0.3 0"/>
-  </xacro:fls_camera>
-  -->
   <xacro:forward_looking_sonar
       namespace="${namespace}"
@@ -63,10 +52,4 @@
     </gazebo>
   </xacro:rexrov_base>
-  <!--xacro:forward_multibeam_p900 namespace="$(arg namespace)" parent_link="$(arg namespace)/base_link">
-    <origin xyz="1.4 0 0.65" rpy="0 0 0"/>
-  </xacro:forward_multibeam_p900-->
-  <!--<xacro:fl_multibeam_generic namespace="$(arg namespace)" parent_link="$(arg namespace)/base_link">
-    <origin xyz="1.4 0 0.65" rpy="0 0 0"/>
-  </xacro:fl_multibeam_generic>-->
   <!-- Joint state publisher plugin -->
   <xacro:default_joint_state_publisher namespace="$(arg namespace)" update_rate="50"/>

Commit message: Cleaned up additonal bugs due to messages produced by branch merge from master on 7/1/2020. Should be working fine now.

File: uuv_descriptions/robots/rexrov_test.xacro (robot description, xacro)
@@ -19,18 +19,4 @@
   <xacro:include filename="$(find uuv_descriptions)/urdf/rexrov_base.xacro"/>
   <xacro:include filename="$(find uuv_descriptions)/urdf/rexrov.gazebo.xacro"/>
-<<<<<<< HEAD
-  <!--xacro:default_camera namespace="${namespace}" parent_link="${namespace}/base_link" suffix="top">
-    <origin xyz="7.5 0 15" rpy="0 1.52 0"/>
-  </xacro:default_camera-->
-  <!--<xacro:uw_depth_camera namespace="${namespace}" parent_link="${namespace}/base_link" suffix="depth">
-    <origin xyz="1.15 0.5 0.4" rpy="0 0.1 0"/>
-  </xacro:uw_depth_camera>-->
-  <!--
-  <xacro:fls_camera namespace="${namespace}" parent_link="${namespace}/base_link" suffix="fls">
-    <origin xyz="1.15 0.5 0.4" rpy="0 0.3 0"/>
-  </xacro:fls_camera>
-  -->
-=======
->>>>>>> realistic-sonar-sim-48
   <xacro:forward_looking_sonar
       namespace="${namespace}"
@@ -66,13 +52,4 @@
     </gazebo>
   </xacro:rexrov_base>
-<<<<<<< HEAD
-  <!--xacro:forward_multibeam_p900 namespace="$(arg namespace)" parent_link="$(arg namespace)/base_link">
-    <origin xyz="1.4 0 0.65" rpy="0 0 0"/>
-  </xacro:forward_multibeam_p900-->
-  <!--<xacro:fl_multibeam_generic namespace="$(arg namespace)" parent_link="$(arg namespace)/base_link">
-    <origin xyz="1.4 0 0.65" rpy="0 0 0"/>
-  </xacro:fl_multibeam_generic>-->
-=======
->>>>>>> realistic-sonar-sim-48
   <!-- Joint state publisher plugin -->
   <xacro:default_joint_state_publisher namespace="$(arg namespace)" update_rate="50"/>

File: uuv_sensor_plugins/uuv_sensor_ros_plugins/urdf/sonar_snippets.xacro (robot description, xacro)
@@ -179,5 +179,5 @@
   <xacro:macro name="forward_looking_sonar"
     params="namespace suffix parent_link topic mass update_rate
-      samples fov width height *inertia *origin">
+      samples fov width height *inertia *origin *visual">
     <!-- Sensor link -->
     <link name="${namespace}/forward_sonar${suffix}_link">
@@ -192,4 +192,5 @@
         </geometry>
       </visual>
+      <!-- <xacro:insert_block name="visual" /> -->
       <xacro:no_collision/>
     </link>
@@ -201,5 +202,4 @@
       <axis xyz="1 0 0"/>
     </joint>
-<<<<<<< HEAD
     <gazebo reference="${namespace}/forward_sonar${suffix}_link">
       <sensor name="${namespace}/image_sonar" type="depth">
@@ -227,81 +227,4 @@
       </sensor>
     </gazebo>
-<<<<<<< HEAD
-  <xacro:macro name="forward_looking_sonar"
-    params="namespace suffix parent_link topic mass update_rate
-      samples fov width height *inertia *origin *visual">
-    <!-- Sensor link -->
-    <link name="${namespace}/forward_sonar${suffix}_link">
-      <inertial>
-        <xacro:insert_block name="inertia" />
-        <mass value="${mass}" />
-        <origin xyz="0 0 0" rpy="0 0 0" />
-      </inertial>
-      <visual>
-        <geometry>
-          <mesh filename="file://$(find uuv_sensor_ros_plugins)/meshes/oe14-372.dae" scale="1 1 1"/>
-        </geometry>
-      </visual>
-      <!-- <xacro:insert_block name="visual" /> -->
-      <xacro:no_collision/>
-    </link>
-    <joint name="${namespace}_forward_sonar${suffix}_joint" type="revolute">
-      <xacro:insert_block name="origin" />
-      <parent link="${parent_link}" />
-      <child link="${namespace}/forward_sonar${suffix}_link" />
-      <limit upper="0" lower="0" effort="0" velocity="0" />
-      <axis xyz="1 0 0"/>
-    </joint>
-    <gazebo reference="${namespace}/forward_sonar${suffix}_link">
-      <sensor name="${namespace}/image_sonar" type="depth">
-        <camera>
-          <horizontal_fov>${fov}</horizontal_fov>
-          <image>
-            <width>${width}</width>
-            <height>${height}</height>
-=======
-    <gazebo reference="${namespace}/forward_sonar${suffix}_link">
-      <sensor name="${namespace}/image_sonar" type="depth">
-        <camera>
-		  <horizontal_fov>${fov}</horizontal_fov>
-          <image>
-		    <width>${width}</width>
-		    <height>${height}</height>
->>>>>>> master
-            <format>R8G8B8</format>
-          </image>
-          <clip>
-            <near>0.1</near>
-            <far>17</far>
-          </clip>
-<<<<<<< HEAD
-          <save enabled="false"> <!--Keeping save disabled to avoid filesystem overload -->
-            <path>/tmp/camera</path>
-          </save>
-        </camera>
-	      <plugin filename="libimage_sonar_ros_plugin.so" name="forward_sonar${suffix}_controller">
-		      <topicName>${topic}</topicName>
-          <frameName>forward_sonar${suffix}_optical_frame</frameName>
-        </plugin>
-        <always_on>true</always_on>
-	      <update_rate>${update_rate}</update_rate>
-      </sensor>
-    </gazebo>
-=======
->>>>>>> realistic-sonar-sim-48
-=======
-          <save enabled="true">
-            <path>/tmp/camera</path>
-          </save>
-        </camera>
-	    <plugin filename="libimage_sonar_ros_plugin.so" name="forward_sonar${suffix}_controller">
-		  <topicName>${topic}</topicName>
-          <frameName>forward_sonar${suffix}_optical_frame</frameName>
-        </plugin>
-        <always_on>true</always_on>
-	    <update_rate>${update_rate}</update_rate>
-      </sensor>
-    </gazebo>
->>>>>>> master
 	<joint name="${namespace}/forward_sonar${suffix}_joint" type="fixed">
       <origin xyz="0 0 0" rpy="${-pi/2} 0 ${-pi/2}"/>
@@ -309,7 +232,4 @@
       <child link="${namespace}/forward_sonar${suffix}_optical_frame"/>
     </joint>
-<<<<<<< HEAD
-=======
->>>>>>> master
 	<link name="${namespace}/forward_sonar${suffix}_optical_frame"/>
   </xacro:macro>
