Commit message: adding forward_looking_sonar to the .xacro

File: uuv_descriptions/robots/rexrov_sonar.xacro (robot description, xacro)
@@ -35,4 +35,21 @@
     </gazebo>
   </xacro:rexrov_base>
+  <xacro:forward_looking_sonar
+      namespace="$(arg namespace)"
+      suffix="down"
+      parent_link="$(arg namespace)/base_link"
+      topic="forward_sonar"
+      mass="0.015"
+      update_rate="40"
+      samples="100"
+        fov="1.54719755"
+        width="768"
+        height="492">
+      <inertia ixx="0.00001" ixy="0.0" ixz="0.0" iyy="0.00001" iyz="0.0" izz="0.00001" />
+      <!--origin xyz="0.83 0 -0.22" rpy="0 ${0.2*pi} 0" /-->
+      <origin xyz="1.40 0 -0.8" rpy="0 0.3 0"/>
+      <visual>
+      </visual>
+  </xacro:forward_looking_sonar>
   <xacro:forward_multibeam_sonar_m450_130 namespace="$(arg namespace)" parent_link="$(arg namespace)/base_link">
     <origin xyz="1.4 0 0.65" rpy="0 0 0"/>
