Commit message: Modified Brazilian Institute FLSonar implementation to better fit the UUVSim environment. Created new launch file and xacros for the FLSonar implementation. \n\n Launch was able to run however FLSonar and other sensors were unable to render successfully. Need to debug and better put the FLSonar implementation into the UUVSim environmetn

File: uuv_sensor_plugins/uuv_sensor_ros_plugins/urdf/sonar_snippets.xacro (robot description, xacro)
@@ -94,4 +94,28 @@
     </xacro:multibeam_sonar>
   </xacro:macro>
+  <xacro:macro name="fl_multibeam_generic" params="namespace parent_link *origin">
+    <xacro:forward_looking_multibeam_sonar
+      namespace="${namespace}"
+      suffix=""
+      parent_link="${parent_link}"
+      topic="sonar"
+      mass="0.02"
+      update_rate="15"
+      samples="512"
+      fov="1.5708"
+      range_min="1.0"
+      range_max="100.0"
+      range_stddev="0.027"
+      mesh="">
+      <inertia ixx="0.00001" ixy="0.0" ixz="0.0" iyy="0.00001" iyz="0.0" izz="0.00001" />
+      <xacro:insert_block name="origin" />
+      <visual>
+        <geometry>
+          <mesh filename="file://$(find uuv_sensor_ros_plugins)/meshes/p900.dae" scale="1 1 1"/>
+        </geometry>
+      </visual>
+    </xacro:forward_looking_multibeam_sonar>
+  </xacro:macro>
+  <!-- xacro for multibeam_sonar -->
   <xacro:macro name="multibeam_sonar"
     params="namespace suffix parent_link topic mass update_rate
@@ -152,3 +176,53 @@
   </gazebo>
   </xacro:macro>
+  <!-- modified version of Brazilian Institute of Robotic's FLS implementation in Gazebo -->
+  <xacro:macro name="forward_looking_multibeam_sonar"
+    params="namespace suffix parent_link topic mass update_rate
+      samples fov range_min range_max range_stddev mesh
+      *inertia *origin *visual">
+    <!-- Sensor link -->
+    <link name="${namespace}/sonar${suffix}_link">
+      <inertial>
+        <xacro:insert_block name="inertia" />
+        <mass value="${mass}" />
+        <origin xyz="0 0 0" rpy="0 0 0" />
+      </inertial>
+      <xacro:insert_block name="visual" />
+      <xacro:no_collision/>
+    </link>
+    <joint name="${namespace}_sonar${suffix}_joint" type="revolute">
+      <xacro:insert_block name="origin" />
+      <parent link="${parent_link}" />
+      <child link="${namespace}/sonar${suffix}_link" />
+      <limit upper="0" lower="0" effort="0" velocity="0" />
+      <axis xyz="1 0 0"/>
+    </joint>
+    <gazebo reference="${namespace}/sonar${suffix}_link">
+      <sensor name='FLSonar' type='camera'>
+        <plugin name="SonarVisual" filename="libuuv_gazebo_ros_flsonar_plugin.so" >
+            <topic>${topic}</topic>
+            <debug>1</debug>
+            <link_reference>${namespace}/sonar${suffix}_link</link_reference>
+            <horizontal_fov>${fov}</horizontal_fov>
+            <vfov>${fov}</vfov>
+            <bin_count>720</bin_count>
+            <beam_count>720</beam_count>
+            <image>
+                <width>720</width>
+                <height>720</height>
+                <format>RGB_FLOAT32</format>
+            </image>
+            <clip>
+                <near>1</near>
+                <far>5</far>
+            </clip>
+            <noise>
+                <type>gaussian</type>
+                <mean>0.0</mean>
+                <stddev>0.1</stddev>
+            </noise>
+        </plugin>
+      </sensor>
+    </gazebo>
+  </xacro:macro>
 </robot>

Commit message: Cleaned up all library, source, and msg files that were completely not used for Nils Bore's FLS sonar implementation

File: uuv_sensor_plugins/uuv_sensor_ros_plugins/urdf/sonar_snippets.xacro (robot description, xacro)
@@ -177,54 +177,4 @@
   </gazebo>
   </xacro:macro>
-  <!-- modified version of Brazilian Institute of Robotic's FLS implementation in Gazebo -->
-  <xacro:macro name="forward_looking_multibeam_sonar"
-    params="namespace suffix parent_link topic mass update_rate
-      samples fov range_min range_max range_stddev mesh
-      *inertia *origin *visual">
-    <!-- Sensor link -->
-    <link name="${namespace}/sonar${suffix}_link">
-      <inertial>
-        <xacro:insert_block name="inertia" />
-        <mass value="${mass}" />
-        <origin xyz="0 0 0" rpy="0 0 0" />
-      </inertial>
-      <xacro:insert_block name="visual" />
-      <xacro:no_collision/>
-    </link>
-    <joint name="${namespace}_sonar${suffix}_joint" type="revolute">
-      <xacro:insert_block name="origin" />
-      <parent link="${parent_link}" />
-      <child link="${namespace}/sonar${suffix}_link" />
-      <limit upper="0" lower="0" effort="0" velocity="0" />
-      <axis xyz="1 0 0"/>
-    </joint>
-    <gazebo reference="${namespace}/sonar${suffix}_link">
-      <sensor name='FLSonar' type='camera'>
-        <plugin name="SonarVisual" filename="libuuv_gazebo_ros_flsonar_plugin.so" >
-            <topic>rexrov/FLSonar</topic>
-            <debug>1</debug>
-            <link_reference>${namespace}/sonar${suffix}_link</link_reference>
-            <horizontal_fov>${fov}</horizontal_fov>
-            <vfov>${fov}</vfov>
-            <bin_count>720</bin_count>
-            <beam_count>720</beam_count>
-            <image>
-                <width>720</width>
-                <height>720</height>
-                <format>RGB_FLOAT32</format>
-            </image>
-            <clip>
-                <near>1</near>
-                <far>5</far>
-            </clip>
-            <noise>
-                <type>gaussian</type>
-                <mean>0.0</mean>
-                <stddev>0.1</stddev>
-            </noise>
-        </plugin>
-      </sensor>
-    </gazebo>
-  </xacro:macro>
   <xacro:macro name="forward_looking_sonar"
     params="namespace suffix parent_link topic mass update_rate

Commit message: changes in the sonar_snippets.xacro to connect the sensor to laseScan

File: uuv_sensor_plugins/uuv_sensor_ros_plugins/urdf/sonar_snippets.xacro (robot description, xacro)
@@ -59,5 +59,5 @@
       fov="2.27"
       range_min="1.0"
-      range_max="100.0"
+      range_max="50.0"
       range_stddev="0.027"
       mesh="">
@@ -94,28 +94,4 @@
     </xacro:multibeam_sonar>
   </xacro:macro>
-  <xacro:macro name="fl_multibeam_generic" params="namespace parent_link *origin">
-    <xacro:forward_looking_multibeam_sonar
-      namespace="${namespace}"
-      suffix=""
-      parent_link="${parent_link}"
-      topic="sonar"
-      mass="0.02"
-      update_rate="15"
-      samples="512"
-      fov="1.5708"
-      range_min="1.0"
-      range_max="100.0"
-      range_stddev="0.027"
-      mesh="">
-      <inertia ixx="0.00001" ixy="0.0" ixz="0.0" iyy="0.00001" iyz="0.0" izz="0.00001" />
-      <xacro:insert_block name="origin" />
-      <visual>
-        <geometry>
-          <mesh filename="file://$(find uuv_sensor_ros_plugins)/meshes/p900.dae" scale="1 1 1"/>
-        </geometry>
-      </visual>
-    </xacro:forward_looking_multibeam_sonar>
-  </xacro:macro>
-  <!-- xacro for multibeam_sonar -->
   <xacro:macro name="multibeam_sonar"
     params="namespace suffix parent_link topic mass update_rate
@@ -140,7 +116,6 @@
   </joint>
   <gazebo reference="${namespace}/sonar${suffix}_link">
-    <sensor type="gpu_ray" name="sonar${suffix}">
+    <sensor type="ray" name="sonar${suffix}">
       <pose>0 0 0 0 0 0</pose>
-      <!--Change value here to make sonar beams visible or not-->
       <visualize>true</visualize>
       <update_rate>${update_rate}</update_rate>
@@ -165,5 +140,5 @@
         </noise>
       </ray>
-      <plugin name="sonar${suffix}_controller" filename="libgazebo_ros_gpu_laser.so">
+      <plugin name="sonar${suffix}_controller" filename="libgazebo_ros_laser.so">
         <topicName>${topic}</topicName>
         <frameName>sonar${suffix}_link</frameName>
@@ -177,60 +152,3 @@
   </gazebo>
   </xacro:macro>
-  <xacro:macro name="forward_looking_sonar"
-    params="namespace suffix parent_link topic mass update_rate
-      samples fov width height *inertia *origin *visual">
-    <!-- Sensor link -->
-    <link name="${namespace}/forward_sonar${suffix}_link">
-      <inertial>
-        <xacro:insert_block name="inertia" />
-        <mass value="${mass}" />
-        <origin xyz="0 0 0" rpy="0 0 0" />
-      </inertial>
-      <visual>
-        <geometry>
-          <mesh filename="file://$(find uuv_sensor_ros_plugins)/meshes/oe14-372.dae" scale="1 1 1"/>
-        </geometry>
-      </visual>
-      <!-- <xacro:insert_block name="visual" /> -->
-      <xacro:no_collision/>
-    </link>
-    <joint name="${namespace}_forward_sonar${suffix}_joint" type="revolute">
-      <xacro:insert_block name="origin" />
-      <parent link="${parent_link}" />
-      <child link="${namespace}/forward_sonar${suffix}_link" />
-      <limit upper="0" lower="0" effort="0" velocity="0" />
-      <axis xyz="1 0 0"/>
-    </joint>
-    <gazebo reference="${namespace}/forward_sonar${suffix}_link">
-      <sensor name="${namespace}/image_sonar" type="depth">
-        <camera>
-          <horizontal_fov>${fov}</horizontal_fov>
-          <image>
-            <width>${width}</width>
-            <height>${height}</height>
-            <format>R8G8B8</format>
-          </image>
-          <clip>
-            <near>0.1</near>
-            <far>17</far>
-          </clip>
-          <save enabled="false"> <!--Keeping save disabled to avoid filesystem overload -->
-            <path>/tmp/camera</path>
-          </save>
-        </camera>
-	      <plugin filename="libimage_sonar_ros_plugin.so" name="forward_sonar${suffix}_controller">
-		      <topicName>${topic}</topicName>
-          <frameName>forward_sonar${suffix}_optical_frame</frameName>
-        </plugin>
-        <always_on>true</always_on>
-	      <update_rate>${update_rate}</update_rate>
-      </sensor>
-    </gazebo>
-	<joint name="${namespace}/forward_sonar${suffix}_joint" type="fixed">
-      <origin xyz="0 0 0" rpy="${-pi/2} 0 ${-pi/2}"/>
-      <parent link="${namespace}/forward_sonar${suffix}_link"/>
-      <child link="${namespace}/forward_sonar${suffix}_optical_frame"/>
-    </joint>
-	<link name="${namespace}/forward_sonar${suffix}_optical_frame"/>
-  </xacro:macro>
 </robot>

Commit message: adding the laserscan as a ray sonar

File: uuv_sensor_plugins/uuv_sensor_ros_plugins/urdf/sonar_snippets.xacro (robot description, xacro)
@@ -59,5 +59,5 @@
       fov="2.27"
       range_min="1.0"
-      range_max="50.0"
+      range_max="100.0"
       range_stddev="0.027"
       mesh="">
@@ -94,4 +94,28 @@
     </xacro:multibeam_sonar>
   </xacro:macro>
+  <xacro:macro name="fl_multibeam_generic" params="namespace parent_link *origin">
+    <xacro:forward_looking_multibeam_sonar
+      namespace="${namespace}"
+      suffix=""
+      parent_link="${parent_link}"
+      topic="sonar"
+      mass="0.02"
+      update_rate="15"
+      samples="512"
+      fov="1.5708"
+      range_min="1.0"
+      range_max="100.0"
+      range_stddev="0.027"
+      mesh="">
+      <inertia ixx="0.00001" ixy="0.0" ixz="0.0" iyy="0.00001" iyz="0.0" izz="0.00001" />
+      <xacro:insert_block name="origin" />
+      <visual>
+        <geometry>
+          <mesh filename="file://$(find uuv_sensor_ros_plugins)/meshes/p900.dae" scale="1 1 1"/>
+        </geometry>
+      </visual>
+    </xacro:forward_looking_multibeam_sonar>
+  </xacro:macro>
+  <!-- xacro for multibeam_sonar -->
   <xacro:macro name="multibeam_sonar"
     params="namespace suffix parent_link topic mass update_rate
@@ -116,6 +140,8 @@
   </joint>
   <gazebo reference="${namespace}/sonar${suffix}_link">
+    <!--<sensor type="gpu_ray" name="sonar${suffix}"> -->
     <sensor type="ray" name="sonar${suffix}">
       <pose>0 0 0 0 0 0</pose>
+      <!--Change value here to make sonar beams visible or not-->
       <visualize>true</visualize>
       <update_rate>${update_rate}</update_rate>
@@ -140,5 +166,6 @@
         </noise>
       </ray>
-      <plugin name="sonar${suffix}_controller" filename="libgazebo_ros_laser.so">
+      <!--<plugin name="sonar${suffix}_controller" filename="libgazebo_ros_gpu_laser.so">-->
+        <plugin name="sonar${suffix}_controller" filename="libgazebo_ros_laser.so">
         <topicName>${topic}</topicName>
         <frameName>sonar${suffix}_link</frameName>
@@ -152,3 +179,60 @@
   </gazebo>
   </xacro:macro>
+  <xacro:macro name="forward_looking_sonar"
+    params="namespace suffix parent_link topic mass update_rate
+      samples fov width height *inertia *origin *visual">
+    <!-- Sensor link -->
+    <link name="${namespace}/forward_sonar${suffix}_link">
+      <inertial>
+        <xacro:insert_block name="inertia" />
+        <mass value="${mass}" />
+        <origin xyz="0 0 0" rpy="0 0 0" />
+      </inertial>
+      <visual>
+        <geometry>
+          <mesh filename="file://$(find uuv_sensor_ros_plugins)/meshes/oe14-372.dae" scale="1 1 1"/>
+        </geometry>
+      </visual>
+      <!-- <xacro:insert_block name="visual" /> -->
+      <xacro:no_collision/>
+    </link>
+    <joint name="${namespace}_forward_sonar${suffix}_joint" type="revolute">
+      <xacro:insert_block name="origin" />
+      <parent link="${parent_link}" />
+      <child link="${namespace}/forward_sonar${suffix}_link" />
+      <limit upper="0" lower="0" effort="0" velocity="0" />
+      <axis xyz="1 0 0"/>
+    </joint>
+    <gazebo reference="${namespace}/forward_sonar${suffix}_link">
+      <sensor name="${namespace}/image_sonar" type="depth">
+        <camera>
+          <horizontal_fov>${fov}</horizontal_fov>
+          <image>
+            <width>${width}</width>
+            <height>${height}</height>
+            <format>R8G8B8</format>
+          </image>
+          <clip>
+            <near>0.1</near>
+            <far>17</far>
+          </clip>
+          <save enabled="false"> <!--Keeping save disabled to avoid filesystem overload -->
+            <path>/tmp/camera</path>
+          </save>
+        </camera>
+	      <plugin filename="libimage_sonar_ros_plugin.so" name="forward_sonar${suffix}_controller">
+		      <topicName>${topic}</topicName>
+          <frameName>forward_sonar${suffix}_optical_frame</frameName>
+        </plugin>
+        <always_on>true</always_on>
+	      <update_rate>${update_rate}</update_rate>
+      </sensor>
+    </gazebo>
+	<joint name="${namespace}/forward_sonar${suffix}_joint" type="fixed">
+      <origin xyz="0 0 0" rpy="${-pi/2} 0 ${-pi/2}"/>
+      <parent link="${namespace}/forward_sonar${suffix}_link"/>
+      <child link="${namespace}/forward_sonar${suffix}_optical_frame"/>
+    </joint>
+	<link name="${namespace}/forward_sonar${suffix}_optical_frame"/>
+  </xacro:macro>
 </robot>
